File: MADI/MADI/trabajo/Tarjeta/Board/Board.kicad_pcb (KiCad board)
At the start: 2 copper layers, 71 x 97 mm, 7 parts, among them J1 Conn_01x10_Female, J2 Conn_01x04_Female, J3 Conn_01x02_Female, J4 Conn_01x08_Female, J5 Conn_01x04_Female, J6 Conn_01x02_Female

Commit message: datos de la PCB
Parts:
- moved J3 62.3 mm to (141.0, 77.5), turned to 0 degrees
Connections:
- net Net-(B1-Pad1) renamed GND
- J2 pad 4: Net-(B1-Pad12) -> Net-(B1-Pad11)
- J3 pad 2: Net-(B1-Pad28) -> Net-(B1-Pad12)
Routing:
- net GND: track 228.2 -> 334.7 mm, vias 2 -> 0
- net Net-(B1-Pad28): track 31.4 -> 0.00 mm
- net Net-(B1-Pad36): track 91.3 -> 67.5 mm
- net Net-(B1-Pad15): track 42.4 -> 59.8 mm
- net Net-(B1-Pad11): track 0.00 -> 12.3 mm
- net Net-(B1-Pad12): track 13.8 -> 18.0 mm
- net Net-(B1-Pad16): track 38.8 -> 42.8 mm
- net Net-(B1-Pad30): track 51.9 -> 54.3 mm, vias 0 -> 2
- net Net-(B1-Pad7): track 66.5 -> 68.4 mm
- net Net-(B1-Pad8): track 62.9 -> 64.1 mm
- net Net-(B1-Pad33): track 61.3 -> 62.5 mm
- net Net-(B1-Pad32): track 58.1 -> 58.9 mm
- net Net-(B1-Pad35): track 35.5 -> 36.2 mm
- added copper zone on B.Cu, net GND
- added copper zone on F.Cu, net GND
