File: MADI/MADI/trabajo/Tarjeta/Board/Board.sch (KiCad schematic (older format))
At the start: 7 parts, among them J1 Conn_01x10_Female, J2 Conn_01x04_Female, J3 Conn_01x02_Female, J4 Conn_01x08_Female, J5 Conn_01x04_Female, J6 Conn_01x02_Female

Commit message: ghgf
Parts:
- J1: footprint (none) -> Connector_PinHeader_2.54mm:PinHeader_1x10_P2.54mm_Vertical
Connections:
- net at B1.30 (15): now also J1.1 (Pin_1); no longer J1.4 (Pin_4)
- net at B1.31 (2): now also J1.2 (Pin_2); no longer J1.3 (Pin_3)
- net at B1.32 (0): now also J1.3 (Pin_3); no longer J1.2 (Pin_2)
- net at B1.33 (4): now also J1.4 (Pin_4); no longer J1.1 (Pin_1)
Changed lines of the file:
@@
 F 0 "J1" H 2792 3175 50  0000 C CNN
 F 1 "Conn_01x10_Female" H 2792 3266 50  0000 C CNN
-F 2 "" H 2900 3900 50  0001 C CNN
+F 2 "Connector_PinHeader_2.54mm:PinHeader_1x10_P2.54mm_Vertical" H 2900 3900 50  0001 C CNN
 F 3 "~" H 2900 3900 50  0001 C CNN
 	1    2900 3900
@@
 	4600 3850 4700 3850
 Wire Wire Line
-	3750 4000 3750 5000
-Wire Wire Line
-	3750 5000 5850 5000
-Wire Wire Line
-	5850 5000 5850 3450
-Wire Wire Line
-	5850 3450 5700 3450
-Wire Wire Line
-	3100 4000 3750 4000
-Wire Wire Line
 	5900 3600 5900 3850
-Wire Wire Line
-	5700 3550 5950 3550
-Wire Wire Line
-	5950 3550 5950 5100
-Wire Wire Line
-	5950 5100 3700 5100
-Wire Wire Line
-	3700 5100 3700 4100
-Wire Wire Line
-	3700 4100 3100 4100
-Wire Wire Line
-	3100 4200 3600 4200
-Wire Wire Line
-	3600 4200 3600 5150
-Wire Wire Line
-	3600 5150 6050 5150
-Wire Wire Line
-	6050 5150 6050 3650
-Wire Wire Line
-	6050 3650 5700 3650
-Wire Wire Line
-	5700 3750 6200 3750
-Wire Wire Line
-	6200 3750 6200 5300
-Wire Wire Line
-	6200 5300 3100 5300
-Wire Wire Line
-	3100 5300 3100 4300
 NoConn ~ 4700 4350
 NoConn ~ 4700 4250
@@
 Wire Wire Line
 	6450 4150 6100 4150
+Wire Wire Line
+	3100 4000 3600 4000
+Wire Wire Line
+	3600 4000 3600 5000
+Wire Wire Line
+	3600 5000 5850 5000
+Wire Wire Line
+	5850 5000 5850 3750
+Wire Wire Line
+	5850 3750 5700 3750
+Wire Wire Line
+	3100 4100 3550 4100
+Wire Wire Line
+	3550 4100 3550 5050
+Wire Wire Line
+	3550 5050 5950 5050
+Wire Wire Line
+	5950 5050 5950 3650
+Wire Wire Line
+	5950 3650 5700 3650
+Wire Wire Line
+	3500 4200 3500 5150
+Wire Wire Line
+	3500 5150 6050 5150
+Wire Wire Line
+	6050 5150 6050 3550
+Wire Wire Line
+	6050 3550 5700 3550
+Wire Wire Line
+	3100 4200 3500 4200
+Wire Wire Line
+	3100 4300 3400 4300
+Wire Wire Line
+	3400 4300 3400 5200
+Wire Wire Line
+	3400 5200 6150 5200
+Wire Wire Line
+	6150 5200 6150 3450
+Wire Wire Line
+	6150 3450 5700 3450
 $EndSCHEMATC

Commit message: datos de la PCB
Parts:
- B1: symbol SparkFun-Boards:ESP32_THING_W_ANT_KEEPOUT -> Board-rescue:ESP32_THING_W_ANT_KEEPOUT-SparkFun-Boards
Connections:
- net GND: now reaches B1.1 (GND), B1.21 (GND), B1.37 (GND), B1.4 (GND), B1.40 (GND), J2.2 (Pin_2), J3.1 (Pin_1), J4.2 (Pin_2), J5.1 (Pin_1), J6.2 (Pin_2)
- net at B1.11 (26): now also J2.4 (Pin_4)
- net at B1.12 (25): now also J3.2 (Pin_2); no longer J2.4 (Pin_4)
- net at B1.28 (18): no longer J3.2 (Pin_2)
Changed lines of the file:
@@
 EESchema Schematic File Version 4
+LIBS:Board-cache
 EELAYER 30 0
 EELAYER END
@@
 $EndDescr
 $Comp
-L SparkFun-Boards:ESP32_THING_W_ANT_KEEPOUT B1
+L Board-rescue:ESP32_THING_W_ANT_KEEPOUT-SparkFun-Boards B1
 U 1 1 5EBFF6FD
 P 5200 3550
@@
 	4700 4150 4400 4150
 Wire Wire Line
-	4400 4150 4400 4600
+	4400 4150 4400 4300
 Wire Wire Line
 	7000 3500 6100 3500
@@
 	5900 3850 5700 3850
 Wire Wire Line
-	4050 2750 4450 2750
-Wire Wire Line
-	4450 2750 4450 3350
-Wire Wire Line
-	4450 3350 4700 3350
-Wire Wire Line
 	4050 2950 4400 2950
 Wire Wire Line
@@
 NoConn ~ 4700 3150
 NoConn ~ 4700 3250
-Wire Wire Line
-	5700 3250 5800 3250
-Wire Wire Line
-	5800 3250 5800 4850
-Wire Wire Line
-	5800 4850 4100 4850
-Wire Wire Line
-	4100 4850 4100 3850
-Wire Wire Line
-	4100 3850 4050 3850
 $Comp
 L Connector:Conn_01x10_Female J1
@@
 	4700 3050 4150 3050
 Wire Wire Line
-	4150 3050 4150 3500
-Wire Wire Line
 	4150 3500 3100 3500
 Wire Wire Line
@@
 	6300 4050 5700 4050
 NoConn ~ 4700 3950
-NoConn ~ 4700 3450
 Wire Wire Line
 	5700 2550 5750 2550
@@
 Wire Wire Line
 	6150 3450 5700 3450
+NoConn ~ 5700 3250
+Wire Wire Line
+	4150 3050 4150 3500
+Wire Wire Line
+	4700 3350 4250 3350
+Wire Wire Line
+	4250 3350 4250 3850
+Wire Wire Line
+	4250 3850 4050 3850
+Wire Wire Line
+	4700 3450 4100 3450
+Wire Wire Line
+	4100 3450 4100 2750
+Wire Wire Line
+	4100 2750 4050 2750
+$Comp
+L power:GND #PWR0101
+U 1 1 5ECF0132
+P 4000 4300
+F 0 "#PWR0101" H 4000 4050 50  0001 C CNN
+F 1 "GND" H 4005 4127 50  0000 C CNN
+F 2 "" H 4000 4300 50  0001 C CNN
+F 3 "" H 4000 4300 50  0001 C CNN
+	1    4000 4300
+	1    0    0    -1
+$EndComp
+Wire Wire Line
+	4000 4300 4400 4300
+Connection ~ 4400 4300
+Wire Wire Line
+	4400 4300 4400 4600
 $EndSCHEMATC

Commit message: hola
Hola
Parts:
- J1: value Conn_01x10_Female -> TouchPad
- J2: value Conn_01x04_Female -> NeoPixel
- J3: value Conn_01x02_Female -> BUZZER
- J4: value Conn_01x08_Female -> MPU6050
- J5: value Conn_01x04_Female -> HC-SR04
- J6: value Conn_01x02_Female -> Alimentacion 5V Externa
Connections:
- net Touch7: now reaches B1.10 (27), J1.8 (Pin_8)
- net Neo: now reaches B1.11 (26), J2.4 (Pin_4)
- net BUZZER: now reaches B1.12 (25), J3.2 (Pin_2)
- net Touch8: now reaches B1.15 (33), J1.9 (Pin_9)
- net Touch9: now reaches B1.16 (32), J1.10 (Pin_10)
- net SDA: now reaches B1.22 (21), J4.4 (Pin_4)
- net SCL: now reaches B1.25 (22), J4.3 (Pin_3)
- net Touch3: now reaches B1.30 (15), J1.1 (Pin_1)
- net Touch2: now reaches B1.31 (2), J1.2 (Pin_2)
- net Touch1: now reaches B1.32 (0), J1.3 (Pin_3)
- net Touch0: now reaches B1.33 (4), J1.4 (Pin_4)
- net ECHO: now reaches B1.34 (17), J5.2 (Pin_2)
- net TRIG: now reaches B1.35 (16), J5.3 (Pin_3)
- net VCC_3: now reaches B1.36 (3V3), B1.5 (3V3), J4.1 (Pin_1)
- net Touch4: now reaches B1.7 (13), J1.5 (Pin_5)
- net Touch5: now reaches B1.8 (12), J1.6 (Pin_6)
- net Touch6: now reaches B1.9 (14), J1.7 (Pin_7)
- net VCC_5: now reaches J2.3 (Pin_3), J5.4 (Pin_4), J6.1 (Pin_1)
Other:
- moved on the sheet: J1, J2, J3, J4, J5, J6
